File: Eagle_Files/AVR_Board_programmer.brd (EAGLE design)
At the start: 38.1 x 46.5 mm, 61 parts, among them J1 SFW24R-1STE1LF, U1 ATMEGA48PA-MMHR28M1-L, U2 MCP6001T-I/OTSOT-23-5_MC-L, U3 LM358PWRDFN-8

Commit message: pulled latest fixes from master
Parts:
- removed 5V, MISO, MOSI, RST, SCK: TPTP13SQ, PiezoFFC:TP13SQ
- removed ADJ+, ADJ-, A_OUT: TPTP10R, PiezoFFC:TP10R
- removed C3: 1uF, PiezoFFC:CAPC1609X80
- removed D2, D3, D4, D5, ERR, TRG: (no value), PiezoFFC:SEEED-LED_LED-0603
- removed D8: BAV199, PiezoFFC:SOT23
- removed E0: C-GRID-04-70553, PiezoFFC:70553-04
- removed FAN0, FAN1, PZ1, TH0: CON-MOLEX-2P-1.27MM048, PiezoFFC:53048-02
- removed HE0: JST-2.54-2X2JST-DUPONT-2.54-2X2, PiezoFFC:HDRRAR4W64P254_2X2_556X736X556B
- removed INT, SS: TPTP06R, testpad:TP06R
- removed R10: 10K, PiezoFFC:R0402
- removed R11, R7: 220R, PiezoFFC:R0402
- removed R12, R5: 330R, PiezoFFC:R0402
- removed R13: 100R, PiezoFFC:R0402
- removed R14: 0R, PiezoFFC:SEEED-RESISTOR_R0603
- removed R15: 680R, PiezoFFC:R0402
- removed R17: 3.3K, PiezoFFC:R0402
- removed R19: 1M, PiezoFFC:R0402
- removed R6: (no value), PiezoFFC:R0402
- removed R9: 470R, PiezoFFC:R0402
- removed SCL, SDA, ⏚: TPTP13SQ, testpad:TP13SQ
- removed U2: MCP6001T-I/OTSOT-23-5_MC-L, PiezoFFC:SOT-23-5_MC-L
- removed U3: LM358PWRDFN-8, PiezoFFC:SON50P200X200X60-9N
- added RESET: (no value), PiezoFFC:SEEED-SWITCH_SW2-2.6-3.0X2.5X1.2+0.4MM
- added RX, TX: (no value), PiezoFFC:SEEED-LED_LED-0603
- added TTL: JST-2.54MM_5P-2.54JST_2.54MM_5P_F, PiezoFFC:HDRVR5W64P254_1X5_1270X254X575B
- added U$2: (no value), PiezoFFC:LOGO-PYR0BALL-SS-20MM
- +5V, GND, RST., RXD, TXD: value TPTP13SQ -> TP; device testpad:TP13SQ -> PiezoFFC:TP13SQ-HOLE
- D1: value 1N4148DFN-1006-2 -> SP0503BAHTG; device PiezoFFC:DIOC1006X70 -> PiezoFFC:SOT143
- J1: value SFW24R-1STE1LF -> 10118192-0001LF; device PiezoFFC:CON24_1X24_DRB_SFW -> PiezoFFC:AMPHENOL_10118192-0001LF
- R1: value 1M -> 22K
- R2: value 10K -> 47K
- R3, R8: value 1K -> (none)
- U1: value ATMEGA48PA-MMHR28M1-L -> CP2102N-A01-GQFN28; device PiezoFFC:28M1-L -> PiezoFFC:QFN50P500X500X80-29N
- moved PWR 22.8 mm to (35.9, 34.8), flipped to the top, turned to 45 degrees
- moved R8 18.8 mm to (33.4, 33.0), flipped to the top, turned to 45 degrees
- moved R3 17.7 mm to (33.0, 38.2)
- moved J1 17.2 mm to (22.7, 13.1), turned to 45 degrees
- moved D1 16.5 mm to (25.8, 21.1), turned to 135 degrees
- moved C1 13.7 mm to (15.0, 22.0), flipped to the top, turned to 180 degrees
- moved C2 10.9 mm to (16.4, 19.9), flipped to the bottom, turned to 45 degrees
- moved R4 10.1 mm to (13.0, 22.0), turned to 90 degrees
- moved R2 9.45 mm to (13.9, 17.9), flipped to the bottom, turned to 180 degrees
- moved R1 8.85 mm to (14.3, 19.4), flipped to the bottom, turned to 270 degrees
- moved U$1 4.51 mm to (18.4, 28.0), flipped to the top, turned to 270 degrees
- moved U1 1.97 mm to (14.4, 24.1), flipped to the bottom, turned to 45 degrees
- moved GND 0.15 mm to (28.5, 32.2)
- moved TXD 0.14 mm to (21.2, 39.3)
- moved +5V 0.11 mm to (24.9, 35.8)
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Connections:
- removed net +5V: +5V.TP, C1.1, D8.2, R10.2, R14.2, R15.1, R3.1, R8.1, U1.16, U1.3, U2.5, U3.8
- removed net COMP-: ADJ+.TP, R1.2, R2.2, U2.1, U3.2
- removed net E0_1A: E0.3, J1.5, J1.6
- removed net E0_1B: E0.4, J1.7, J1.8
- removed net E0_2A: E0.2, J1.3, J1.4
- removed net E0_2B: E0.1, J1.1, J1.2
- removed net ERR_LED: ERR.+, U1.1
- removed net FAN0_GATE: D5.-, FAN0.1, J1.17
- removed net FAN1_GATE: D4.-, FAN1.1, J1.15
- removed net GAIN_FB: R17.2, R2.1, U2.4
- removed net HE0-: D3.-, HE0.3, HE0.4, J1.21, J1.22
- removed net PZ+: D8.3, PZ1.2, R19.2, U2.3
- removed net PZ_AMP_OUT: A_OUT.TP, R13.1, U3.1
- removed net SCL: SCL.TP, U1.24
- removed net SDA: SDA.TP, U1.23
- removed net SPI_MISO: MISO.TP, U1.14
- removed net SPI_MOSI: MOSI.TP, U1.13
- removed net SPI_SCK: SCK.TP, U1.15
- removed net SPI_SS: SS.TP, U1.12
- removed net TH0+: J1.20, TH0.1
- removed net TH0-: J1.19, TH0.2
- removed net TRG_LED: D2.+, R6.2, TRG.+
- removed net TTL_RXD: RXD.TP, U1.26
- removed net TTL_TXD: TXD.TP, U1.27
- removed net VADJ_R0: R11.2, R7.1, U1.5
- removed net VADJ_R1: R11.1, R12.2, U1.6
- removed net VADJ_R2: R12.1, R5.2, U1.7
- removed net VADJ_R3: R5.1, R9.2, U1.8
- removed net VADJ_SENSE: ADJ-.TP, R15.2, R7.2, U1.20, U3.3
- removed net VCC: HE0.1, HE0.2, J1.23, J1.24
- removed net VCC_REG: 5V.TP, C2.2, D1.C, J1.9, R14.1
- removed net VREF_IN: R10.1, R4.2, U3.5
- removed net V_FOLLOW: R1.1, U1.19, U3.6, U3.7
- removed net V_INT: C3.1, FAN0.2, FAN1.2, J1.10, J1.11
- removed net Z_MIN_TRIG: J1.13, R6.1, U1.11
- removed net Z_TRG: INT.TP, R13.2, U1.28
- new net 5V_DC: +5V.TP, C2.2, D1.2, J1.1, R1.2, R3.1, R8.1, TTL.1, U1.7
- new net D+: D1.4, J1.3, U1.4
- new net D-: D1.3, J1.2, U1.5
- new net PGM_RST: C1.2, R4.2, U1.28
- new net RXD: RXD.TP, TTL.4, U1.26
- new net RXT: RX.-, U1.19
- new net TXD: TTL.3, TXD.TP, U1.25
- new net TXT: TX.-, U1.18
- new net VBUS: R1.1, R2.2, R4.1, TTL.5, U1.8
- new net VDD: U1.6
- net GND: now also D1.1, J1.5, J1.SH1, J1.SH2, J1.SH3, J1.SH4, J1.SH5, J1.SH6, R2.1, RESET.1, TTL.2, U1.3; no longer C1.2, C3.2, D1.A, D2.-, D8.1, ERR.-, J1.12, J1.14, J1.16, J1.18, J1.25, J1.26, PZ1.1, R17.1, R19.1, R4.1, R9.1, TRG.-, U1.18, U1.4, U2.2, U3.4, ⏚.TP
- net LED_VCC: now also RX.+, TX.+; no longer D3.+, D4.+, D5.+
- net RST: now also C1.1, RESET.2; no longer RST.TP, U1.25
Routing:
- net 5V_DC: track 0.00 -> 68.3 mm, vias 0 -> 1
- net +5V: track 68.3 -> 0.00 mm, vias 6 -> 0
- net TRG_LED: track 51.2 -> 0.00 mm, vias 3 -> 0
- net TXD: track 0.00 -> 45.8 mm
- net V_INT: track 40.8 -> 0.00 mm, vias 1 -> 0
- net RXD: track 0.00 -> 40.6 mm
- net TXT: track 0.00 -> 36.2 mm, vias 0 -> 1
- net VCC_REG: track 31.7 -> 0.00 mm, vias 1 -> 0
- net RXT: track 0.00 -> 31.6 mm, vias 0 -> 1
- net RST: track 59.5 -> 29.0 mm, vias 3 -> 0
- net LED_VCC: track 29.1 -> 3.03 mm
- net SPI_MOSI: track 25.8 -> 0.00 mm, vias 3 -> 0
- net SPI_SCK: track 25.7 -> 0.00 mm, vias 3 -> 0
- net FAN1_GATE: track 24.1 -> 0.00 mm
- net SPI_MISO: track 22.8 -> 0.00 mm, vias 3 -> 0
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Other:
- board size 38.1 x 46.5 mm -> 39.6 x 46.5 mm
- board text added: "- +"
- board text removed: "+ -"
- board text removed: "2B 2A 1A 1B"
- board text removed: "Fan0"
- board text removed: "Fan1"
- board text removed: "HE0"
- board text removed: "PZ1"
- board text removed: "TH0"
